Commit message: Stereo Vision api created

File: pandaqb_movegroup_control/urdf/pandaqb_description.urdf.xacro (robot description, xacro)
@@ -12,6 +12,6 @@
     <!-- Import the QB Hand and connect it to the created link -->
     <xacro:include filename="$(find qb_hand_description)/urdf/qbhand.utils.xacro"/>
-    <xacro:build_hand_from_yaml configuration="qbhand_right" namespace="qbhand" parent="panda_qb">
-        <origin xyz="0 0 0" rpy="0 0 0"/>
-    </xacro:build_hand_from_yaml>
+	<xacro:build_hand_2m_from_yaml configuration="qbhand_right" namespace="qbhand2m" parent="panda_qb">
+		<origin xyz="0 0 0" rpy="0 0 0"/>
+	</xacro:build_hand_2m_from_yaml>
 </robot>
