Commit message: some calibration things

File: movit_config_only_panda/config/gazebo_panda.urdf (robot description, URDF)
Before this commit: robot panda, 17 links, 16 joints
Links:
- link panda_link0: geometry collision mesh filename=package://panda_qb_description_control/meshes/collision/lin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; visual mesh filename=package://panda_qb_description_control/meshes/visual/link0.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
- link panda_link1: geometry collision mesh filename=package://panda_qb_description_control/meshes/collision/lin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; visual mesh filename=package://panda_qb_description_control/meshes/visual/link1.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
- link panda_link2: geometry collision mesh filename=package://panda_qb_description_control/meshes/collision/lin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; visual mesh filename=package://panda_qb_description_control/meshes/visual/link2.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
- link panda_link3: geometry collision mesh filename=package://panda_qb_description_control/meshes/collision/lin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; visual mesh filename=package://panda_qb_description_control/meshes/visual/link3.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
- link panda_link4: geometry collision mesh filename=package://panda_qb_description_control/meshes/collision/lin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; visual mesh filename=package://panda_qb_description_control/meshes/visual/link4.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
- link panda_link5: geometry collision mesh filename=package://panda_qb_description_control/meshes/collision/lin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; visual mesh filename=package://panda_qb_description_control/meshes/visual/link5.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
- link panda_link6: geometry collision mesh filename=package://panda_qb_description_control/meshes/collision/lin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; visual mesh filename=package://panda_qb_description_control/meshes/visual/link6.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
- link panda_link7: geometry collision mesh filename=package://panda_qb_description_control/meshes/collision/lin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; visual mesh filename=package://panda_qb_description_control/meshes/visual/link7.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

File: movit_config_only_panda/config/gazebo_panda_qb.urdf (robot description, URDF)
Before this commit: robot panda_qb, 19 links, 18 joints
Links:
- removed link panda_qb_link
- added link camera_frame
- link panda_link0: geometry collision mesh filename=package://franka_description/meshes/collision/link0.stl; visual mesh filename=package://franka_description/meshes/visual/link0.dae
- link panda_link1: geometry collision mesh filename=package://franka_description/meshes/collision/link1.stl; visual mesh filename=package://franka_description/meshes/visual/link1.dae
- link panda_link2: geometry collision mesh filename=package://franka_description/meshes/collision/link2.stl; visual mesh filename=package://franka_description/meshes/visual/link2.dae
- link panda_link3: geometry collision mesh filename=package://franka_description/meshes/collision/link3.stl; visual mesh filename=package://franka_description/meshes/visual/link3.dae
- link panda_link4: geometry collision mesh filename=package://franka_description/meshes/collision/link4.stl; visual mesh filename=package://franka_description/meshes/visual/link4.dae
- link panda_link5: geometry collision mesh filename=package://franka_description/meshes/collision/link5.stl; visual mesh filename=package://franka_description/meshes/visual/link5.dae
- link panda_link6: geometry collision mesh filename=package://franka_description/meshes/collision/link6.stl; visual mesh filename=package://franka_description/meshes/visual/link6.dae
- link panda_link7: geometry collision mesh filename=package://franka_description/meshes/collision/link7.stl; visual mesh filename=package://franka_description/meshes/visual/link7.dae
Joints:
- removed joint fixed
- removed joint panda_qb_link__camera_support_link
- added joint camera_joint: type fixed, parent camera_support_link, child camera_frame, origin xyz=0.1 0 0.1 rpy=0 0 0
- added joint panda_support_link__camera_support_link: type fixed, parent panda_link8, child camera_support_link
