Commit message: some launch modifications

File: movit_config_only_panda/config/gazebo_panda_qb.urdf (robot description, URDF)
Before this commit: robot panda, 17 links, 16 joints
Links:
- added link camera_support_link, mass 0.1; collision mesh filename=package://pandaqb_movegroup_control/meshes/camera_support.s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 scale=0.001 0.001 0.001; visual mesh filename=package://pandaqb_movegroup_control/meshes/camera_support.s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 scale=0.001 0.001 0.001
- added link panda_qb_link
Joints:
- added joint fixed: type fixed, parent panda_link8, child panda_qb_link
- added joint panda_qb_link__camera_support_link: type fixed, parent panda_qb_link, child camera_support_link

File: pandaqb_movegroup_control/urdf/pandaqb_description.urdf.xacro (robot description, xacro)
@@ -1,19 +1,7 @@
 <?xml version="1.0"?>
-<robot xmlns:xacro="http://www.ros.org/wiki/xacro">
-    <!-- Import the Franka arm -->
-    <xacro:include filename="$(find franka_description)/robots/common/franka_arm.xacro" />
-    <xacro:franka_arm arm_id="panda" safety_distance="0.03" gazebo="false" joint_limits="${xacro.load_yaml('$(find franka_description)/robots/panda/joint_limits.yaml')}"/>
-    <!-- Create a link and a joint to connect the last link of the panda arm with the base of the qb hand -->
-    <link name="panda_qb_link"/>
-    <joint name="fixed" type="fixed">
-        <parent link="panda_link8"/>
-        <child link="panda_qb_link"/>
-    </joint>
-    <!-- Import the QB Hand and connect it to the created link -->
-    <xacro:include filename="$(find qb_hand_description)/urdf/qbhand.utils.xacro"/>
-	<xacro:build_hand_2m_from_yaml configuration="qbhand_right" namespace="qbhand2m" parent="panda_qb">
-		<origin xyz="0 0 0" rpy="0 0 0"/>
-	</xacro:build_hand_2m_from_yaml>
-    <!-- Import the camera support and connect it to the created link -->
-    <xacro:include filename="$(find pandaqb_movegroup_control)/urdf/AroundSupport.xacro"/>
+<robot xmlns:xacro="http://www.ros.org/wiki/xacro" name="panda_qb">
+  <xacro:include filename="$(find pandaqb_movegroup_control)/urdf/pandaqb_robot.xacro"/>
+  <xacro:qb_panda_robot
+    joint_limits="${xacro.load_yaml('$(find franka_description)/robots/panda/joint_limits.yaml')}">
+  </xacro:qb_panda_robot>
 </robot>

File: pandaqb_movegroup_control/urdf/pandaqb_robot.xacro (robot description, xacro)
@@ -1,75 +1,16 @@
 <?xml version='1.0' encoding='utf-8'?>
 <robot xmlns:xacro="http://www.ros.org/wiki/xacro">
-  <xacro:macro name="qb_franka_robot" params="joint_limits">
-    <!-- Should a qb_gripper be mounted at the flange?" -->
-    <xacro:arg name="hand" default="false" />
-    <!-- Is the robot being simulated in gazebo?" -->
+  <xacro:macro name="qb_panda_robot" params="joint_limits">
     <xacro:arg name="gazebo" default="false" />
-    <xacro:include filename="$(find franka_description)/robots/common/utils.xacro" />
+    <xacro:arg name="hand" default="true" />
     <xacro:include filename="$(find franka_description)/robots/common/franka_arm.xacro" />
     <xacro:franka_arm arm_id="panda" safety_distance="0.03" gazebo="$(arg gazebo)" joint_limits="${joint_limits}"/>
+    <xacro:include filename="$(find pandaqb_movegroup_control)/urdf/camera_support.xacro"/>
     <xacro:if value="$(arg hand)">
-      <!-- Create a link and a joint to connect the last link of the panda arm with the base of the qb hand -->
-      <link name="panda_qb_link"/>
-      <joint name="fixed" type="fixed">
-          <parent link="panda_link8"/>
-          <child link="panda_qb_link"/>
-      </joint>
       <!-- Import the QB Hand and connect it to the created link -->
       <xacro:include filename="$(find qb_hand_description)/urdf/qbhand.utils.xacro"/>
-      <xacro:build_hand_2m_from_yaml configuration="qbhand_right" namespace="qbhand2m" parent="panda_qb">
-        <origin xyz="0 0 0" rpy="0 0 0"/>
+      <xacro:build_hand_2m_from_yaml configuration="qbhand_right" namespace="qbhand2m" parent="camera_support">
+        <origin xyz="0 0 0.01" rpy="0 0 0"/>
       </xacro:build_hand_2m_from_yaml>
-      <xacro:include filename="$(find pandaqb_movegroup_control)/urdf/AroundSupport.xacro"/>
-    </xacro:if>
-    <!-- Define additional Gazebo tags -->
-    <xacro:if value="$(arg gazebo)">
-      <xacro:arg name="xyz" default="0 0 0" />
-      <xacro:arg name="rpy" default="0 0 0" />
-      <!-- Gazebo requires a joint to a link called "world" for statically mounted robots -->
-      <link name="world" />
-      <joint name="world_joint" type="fixed">
-        <origin xyz="$(arg xyz)" rpy="$(arg rpy)" />
-        <parent link="world" />
-        <child  link="panda_link0" />
-      </joint>
-      <!-- <xacro:gazebo-joint joint="panda_joint1" transmission="hardware_interface/PositionJointInterface" />
-      <xacro:gazebo-joint joint="panda_joint2" transmission="hardware_interface/PositionJointInterface" />
-      <xacro:gazebo-joint joint="panda_joint3" transmission="hardware_interface/PositionJointInterface" />
-      <xacro:gazebo-joint joint="panda_joint4" transmission="hardware_interface/PositionJointInterface" />
-      <xacro:gazebo-joint joint="panda_joint5" transmission="hardware_interface/PositionJointInterface" />
-      <xacro:gazebo-joint joint="panda_joint6" transmission="hardware_interface/PositionJointInterface" />
-      <xacro:gazebo-joint joint="panda_joint7" transmission="hardware_interface/PositionJointInterface" />
-      <xacro:gazebo-joint joint="panda_joint1" transmission="hardware_interface/VelocityJointInterface" />
-      <xacro:gazebo-joint joint="panda_joint2" transmission="hardware_interface/VelocityJointInterface" />
-      <xacro:gazebo-joint joint="panda_joint3" transmission="hardware_interface/VelocityJointInterface" />
-      <xacro:gazebo-joint joint="panda_joint4" transmission="hardware_interface/VelocityJointInterface" />
-      <xacro:gazebo-joint joint="panda_joint5" transmission="hardware_interface/VelocityJointInterface" />
-      <xacro:gazebo-joint joint="panda_joint6" transmission="hardware_interface/VelocityJointInterface" />
-      <xacro:gazebo-joint joint="panda_joint7" transmission="hardware_interface/VelocityJointInterface" />
-      <xacro:gazebo-joint joint="panda_joint1" transmission="hardware_interface/EffortJointInterface" />
-      <xacro:gazebo-joint joint="panda_joint2" transmission="hardware_interface/EffortJointInterface" />
-      <xacro:gazebo-joint joint="panda_joint3" transmission="hardware_interface/EffortJointInterface" />
-      <xacro:gazebo-joint joint="panda_joint4" transmission="hardware_interface/EffortJointInterface" />
-      <xacro:gazebo-joint joint="panda_joint5" transmission="hardware_interface/EffortJointInterface" />
-      <xacro:gazebo-joint joint="panda_joint6" transmission="hardware_interface/EffortJointInterface" />
-      <xacro:gazebo-joint joint="panda_joint7" transmission="hardware_interface/EffortJointInterface" /> -->
-      <xacro:transmission-franka-state arm_id="panda" />
-      <xacro:transmission-franka-model arm_id="panda"
-         root="panda_joint1"
-         tip="panda_joint8"
-       />
-      <!-- <xacro:if value="$(arg hand)">
-        <gazebo>
-          <plugin name="qb_hand_gazebo_plugin" filename="libqb_hand_gazebo_plugin.so"/>
-        </gazebo>
-      </xacro:if> -->
-      <!-- <gazebo>
-        <plugin name="gazebo_ros_control" filename="libgazebo_ros_control.so">
-          <controlPeriod>0.001</controlPeriod>
-          <robotSimType>franka_gazebo/FrankaHWSim</robotSimType>
-        </plugin>
-        <self_collide>true</self_collide>
-      </gazebo> -->
     </xacro:if>
   </xacro:macro>

Commit message: some moveit setup

File: movit_config_only_panda/config/gazebo_panda_qb.urdf (robot description, URDF)
Before this commit: robot panda_qb, 19 links, 18 joints
Joints:
- joint camera_joint: origin xyz=0.1 0 0.1 rpy=0 0 0 -> xyz=0.06 0.06 0.02 rpy=0.0872665 0 2.35619

File: panda_qb_description/urdf/camera_support.xacro (robot description, xacro)
@@ -28,5 +28,4 @@
     </inertial>
   </link>
-  <!-- Gazebo requires a joint to a link called "world" for statically mounted robots -->
   <link name="camera_frame" />
   <joint name="camera_joint" type="fixed">

Commit message: upates

File: movit_config_only_panda/config/gazebo_panda_qb.urdf (robot description, URDF)
Before this commit: robot panda_qb, 19 links, 18 joints
Joints:
- joint camera_joint: origin xyz=0.06 0.06 0.02 rpy=0.0872665 0 2.35619 -> xyz=-0.041387 -0.0627379 0.0525437 rpy=3.08447 -3.11784 3.10978; parent camera_support_link -> panda_link8

File: movit_config_panda_qb_5/config/gazebo_panda_qb.urdf (robot description, URDF)
Before this commit: robot panda_qb, 59 links, 58 joints
Joints:
- joint camera_joint: origin xyz=0.06 0.06 0.02 rpy=0.0872665 0 2.35619 -> rpy=3.08447 -3.11784 3.10978; parent qb_hand_wrist_link -> panda_link8

File: movit_panda_gripper/config/gazebo_panda_qb.urdf (robot description, URDF)
Before this commit: robot panda_qb, 24 links, 23 joints
Joints:
- joint camera_joint: origin xyz=0.06 0.06 0.02 rpy=0.0872665 0 2.35619 -> xyz=-0.041387 -0.0627379 0.0525437 rpy=3.08447 -3.11784 3.10978; parent camera_support_link -> panda_link8

File: panda_qb_description/urdf/camera_support.xacro (robot description, xacro)
@@ -28,10 +28,8 @@
     </inertial>
   </link>
-  <link name="camera_frame" />
-  <joint name="camera_joint" type="fixed">
-    <!-- <origin xyz="-0.0414091 -0.0579333 0.0614579" rpy="-0.019865 0.0305123 -0.0144474 0.999233" /> -->
-    <origin xyz="0.06 0.06 0.02" rpy="0.0872665 0 2.35619" />
-    <parent link="camera_support_link" />
+  <!-- <joint name="camera_joint" type="fixed">
+    <origin xyz="-0.041387 -0.0627379 0.0525437" rpy="3.08447 -3.11784 3.10978" />
+    <parent link="panda_link8" />
     <child  link="camera_frame" />
-  </joint>
+  </joint> -->
 </robot>

File: panda_qb_description/urdf/pandaqb_robot.xacro (robot description, xacro)
@@ -15,5 +15,5 @@
     <link name="pinch_link" />
     <joint name="pinch_joint" type="fixed">
-      <origin xyz="0.007 -0.009 0.022" rpy="0.0872665 0 0.523598775" />
+      <origin xyz="-0.0 -0.014 0.022" rpy="0 0 0.523598775" />
       <parent link="qbhand2m1_end_effector_link" />
       <child  link="pinch_link" />
@@ -21,5 +21,5 @@
     <link name="power_link" />
     <joint name="power_joint" type="fixed">
-      <origin xyz="0.01 -0.02 0.0" rpy="0 0 0.523598775" />
+      <origin xyz="0.02 -0.02 -0.005" rpy="0 0 0.523598775" />
       <parent link="qbhand2m1_end_effector_link" />
       <child  link="power_link" />

File: panda_qb_description/urdf/qb_hand_wrist.xacro (robot description, xacro)
@@ -30,6 +30,6 @@
   <link name="camera_frame" />
   <joint name="camera_joint" type="fixed">
-    <origin xyz="-0.0371711 -0.0595898 0.0627352" rpy="3.10255 2.99161 3.10566" />
-    <parent link="qb_hand_wrist_link" />
+    <origin xyz="-0.041387 -0.0627379 0.0525437" rpy="3.08447 -3.11784 3.10978" />
+    <parent link="panda_link8" />
     <child  link="camera_frame" />
   </joint>
