Commit message: hand movegroup can actuate on qb_hand_controllers

File: movit_config_panda_qb_2/config/gazebo_panda_qb.urdf (robot description, URDF)
Before this commit: robot panda_qb, 58 links, 57 joints
Links:
- removed link qbhand2m_base_link
- removed link qbhand2m_end_effector_link
- removed link qbhand2m_index_distal_link
- removed link qbhand2m_index_distal_virtual_link
- removed link qbhand2m_index_knuckle_link
- removed link qbhand2m_index_middle_link
- removed link qbhand2m_index_middle_virtual_link
- removed link qbhand2m_index_proximal_link
- removed link qbhand2m_index_proximal_virtual_link
- removed link qbhand2m_little_distal_link
- removed link qbhand2m_little_distal_virtual_link
- removed link qbhand2m_little_knuckle_link
- removed link qbhand2m_little_middle_link
- removed link qbhand2m_little_middle_virtual_link
- removed link qbhand2m_little_proximal_link
- removed link qbhand2m_little_proximal_virtual_link
- removed link qbhand2m_manipulation_tendon_virtual_link
- removed link qbhand2m_middle_distal_link
- removed link qbhand2m_middle_distal_virtual_link
- removed link qbhand2m_middle_knuckle_link
- removed link qbhand2m_middle_middle_link
- removed link qbhand2m_middle_middle_virtual_link
- removed link qbhand2m_middle_proximal_link
- removed link qbhand2m_middle_proximal_virtual_link
- removed link qbhand2m_motor_1_tendon_virtual_link
- removed link qbhand2m_motor_2_tendon_virtual_link
- removed link qbhand2m_palm_link
- removed link qbhand2m_ring_distal_link
- removed link qbhand2m_ring_distal_virtual_link
- removed link qbhand2m_ring_knuckle_link
- removed link qbhand2m_ring_middle_link
- removed link qbhand2m_ring_middle_virtual_link
- removed link qbhand2m_ring_proximal_link
- removed link qbhand2m_ring_proximal_virtual_link
- removed link qbhand2m_synergy_tendon_virtual_link
- removed link qbhand2m_thumb_distal_link
- removed link qbhand2m_thumb_distal_virtual_link
- removed link qbhand2m_thumb_knuckle_link
- removed link qbhand2m_thumb_proximal_link
- removed link qbhand2m_thumb_proximal_virtual_link
- added link camera_frame
- added link qbhand2m1_base_link, mass 0.45; collision mesh filename=package://qb_hand_description/meshes/flange_iso_04.stl scale=0.001 0.001 0.001; visual mesh filename=package://qb_hand_description/meshes/flange_iso_04.stl scale=0.001 0.001 0.001
- added link qbhand2m1_end_effector_link
- added link qbhand2m1_index_distal_link, mass 0.009; collision mesh filename=package://qb_hand_description/meshes/ph_distal_collision.stl scale=0.001 0.001 0.001; visual mesh filename=package://qb_hand_description/meshes/ph_distal.stl scale=0.001 0.001 0.001
- added link qbhand2m1_index_distal_virtual_link, mass 1e-4
- added link qbhand2m1_index_knuckle_link, mass 0.0095; collision mesh filename=package://qb_hand_description/meshes/ph_knuckle_collision.s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 scale=0.001 0.001 0.001; visual mesh filename=package://qb_hand_description/meshes/ph_knuckle.stl scale=0.001 0.001 0.001
- added link qbhand2m1_index_middle_link, mass 0.0063; collision mesh filename=package://qb_hand_description/meshes/ph_short_collision.stl scale=0.001 0.001 0.001; visual mesh filename=package://qb_hand_description/meshes/ph_short.stl scale=0.001 0.001 0.001
- added link qbhand2m1_index_middle_virtual_link, mass 1e-4
- added link qbhand2m1_index_proximal_link, mass 0.0082; collision mesh filename=package://qb_hand_description/meshes/ph_medium_collision.stl scale=0.001 0.001 0.001; visual mesh filename=package://qb_hand_description/meshes/ph_medium.stl scale=0.001 0.001 0.001
- added link qbhand2m1_index_proximal_virtual_link, mass 1e-4
- added link qbhand2m1_little_distal_link, mass 0.009; collision mesh filename=package://qb_hand_description/meshes/ph_distal_collision.stl scale=0.001 0.001 0.001; visual mesh filename=package://qb_hand_description/meshes/ph_distal.stl scale=0.001 0.001 0.001
- added link qbhand2m1_little_distal_virtual_link, mass 1e-4
- added link qbhand2m1_little_knuckle_link, mass 0.0095; collision mesh filename=package://qb_hand_description/meshes/ph_knuckle_collision.s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 scale=0.001 0.001 0.001; visual mesh filename=package://qb_hand_description/meshes/ph_knuckle.stl scale=0.001 0.001 0.001
- added link qbhand2m1_little_middle_link, mass 0.0063; collision mesh filename=package://qb_hand_description/meshes/ph_short_collision.stl scale=0.001 0.001 0.001; visual mesh filename=package://qb_hand_description/meshes/ph_short.stl scale=0.001 0.001 0.001
- added link qbhand2m1_little_middle_virtual_link, mass 1e-4
- added link qbhand2m1_little_proximal_link, mass 0.0063; collision mesh filename=package://qb_hand_description/meshes/ph_short_collision.stl scale=0.001 0.001 0.001; visual mesh filename=package://qb_hand_description/meshes/ph_short.stl scale=0.001 0.001 0.001
- added link qbhand2m1_little_proximal_virtual_link, mass 1e-4
- added link qbhand2m1_manipulation_tendon_virtual_link, mass 1e-4
- added link qbhand2m1_middle_distal_link, mass 0.009; collision mesh filename=package://qb_hand_description/meshes/ph_distal_collision.stl scale=0.001 0.001 0.001; visual mesh filename=package://qb_hand_description/meshes/ph_distal.stl scale=0.001 0.001 0.001
- added link qbhand2m1_middle_distal_virtual_link, mass 1e-4
- added link qbhand2m1_middle_knuckle_link, mass 0.0095; collision mesh filename=package://qb_hand_description/meshes/ph_knuckle_collision.s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 scale=0.001 0.001 0.001; visual mesh filename=package://qb_hand_description/meshes/ph_knuckle.stl scale=0.001 0.001 0.001
- added link qbhand2m1_middle_middle_link, mass 0.0063; collision mesh filename=package://qb_hand_description/meshes/ph_short_collision.stl scale=0.001 0.001 0.001; visual mesh filename=package://qb_hand_description/meshes/ph_short.stl scale=0.001 0.001 0.001
- added link qbhand2m1_middle_middle_virtual_link, mass 1e-4
- added link qbhand2m1_middle_proximal_link, mass 0.0082; collision mesh filename=package://qb_hand_description/meshes/ph_medium_collision.stl scale=0.001 0.001 0.001; visual mesh filename=package://qb_hand_description/meshes/ph_medium.stl scale=0.001 0.001 0.001
- added link qbhand2m1_middle_proximal_virtual_link, mass 1e-4
- added link qbhand2m1_motor_1_tendon_virtual_link, mass 1e-4
- added link qbhand2m1_motor_2_tendon_virtual_link, mass 1e-4
- added link qbhand2m1_palm_link, mass 0.45; collision mesh filename=package://qb_hand_description/meshes/palm_pinch_r.stl scale=0.001 0.001 0.001; visual mesh filename=package://qb_hand_description/meshes/palm_pinch_r.stl scale=0.001 0.001 0.001
- added link qbhand2m1_ring_distal_link, mass 0.009; collision mesh filename=package://qb_hand_description/meshes/ph_distal_collision.stl scale=0.001 0.001 0.001; visual mesh filename=package://qb_hand_description/meshes/ph_distal.stl scale=0.001 0.001 0.001
- added link qbhand2m1_ring_distal_virtual_link, mass 1e-4
- added link qbhand2m1_ring_knuckle_link, mass 0.0095; collision mesh filename=package://qb_hand_description/meshes/ph_knuckle_collision.s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 scale=0.001 0.001 0.001; visual mesh filename=package://qb_hand_description/meshes/ph_knuckle.stl scale=0.001 0.001 0.001
- added link qbhand2m1_ring_middle_link, mass 0.0063; collision mesh filename=package://qb_hand_description/meshes/ph_short_collision.stl scale=0.001 0.001 0.001; visual mesh filename=package://qb_hand_description/meshes/ph_short.stl scale=0.001 0.001 0.001
- added link qbhand2m1_ring_middle_virtual_link, mass 1e-4
- added link qbhand2m1_ring_proximal_link, mass 0.0082; collision mesh filename=package://qb_hand_description/meshes/ph_medium_collision.stl scale=0.001 0.001 0.001; visual mesh filename=package://qb_hand_description/meshes/ph_medium.stl scale=0.001 0.001 0.001
- added link qbhand2m1_ring_proximal_virtual_link, mass 1e-4
- added link qbhand2m1_synergy_tendon_virtual_link, mass 1e-4
- added link qbhand2m1_thumb_distal_link, mass 0.009; collision mesh filename=package://qb_hand_description/meshes/ph_distal_collision.stl scale=0.001 0.001 0.001; visual mesh filename=package://qb_hand_description/meshes/ph_distal.stl scale=0.001 0.001 0.001
- added link qbhand2m1_thumb_distal_virtual_link, mass 1e-4
- added link qbhand2m1_thumb_knuckle_link, mass 0.01; collision mesh filename=package://qb_hand_description/meshes/ph_thumb_r_collision.s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 scale=0.001 0.001 0.001; visual mesh filename=package://qb_hand_description/meshes/ph_thumb_r.stl scale=0.001 0.001 0.001
- added link qbhand2m1_thumb_proximal_link, mass 0.0063; collision mesh filename=package://qb_hand_description/meshes/ph_short_collision.stl scale=0.001 0.001 0.001; visual mesh filename=package://qb_hand_description/meshes/ph_short.stl scale=0.001 0.001 0.001
- added link qbhand2m1_thumb_proximal_virtual_link, mass 1e-4
- link camera_support_link: geometry collision mesh filename=package://panda_qb_description/meshes/camera_support.stl scale=0.001 0.001 0.001; visual mesh filename=package://panda_qb_description/meshes/camera_support.stl scale=0.001 0.001 0.001
Joints:
- removed joint qbhand2m_base_fixed_joint
- removed joint qbhand2m_d 
- removed joint qbhand2m_end_effector_fixed_joint
- removed joint qbhand2m_index_distal_joint
- removed joint qbhand2m_index_distal_virtual_joint
- removed joint qbhand2m_index_knuckle_joint
- removed joint qbhand2m_index_middle_joint
- removed joint qbhand2m_index_middle_virtual_joint
- removed joint qbhand2m_index_proximal_joint
- removed joint qbhand2m_index_proximal_virtual_joint
- removed joint qbhand2m_little_distal_joint
- removed joint qbhand2m_little_distal_virtual_joint
- removed joint qbhand2m_little_knuckle_joint
- removed joint qbhand2m_little_middle_joint
- removed joint qbhand2m_little_middle_virtual_joint
- removed joint qbhand2m_little_proximal_joint
- removed joint qbhand2m_little_proximal_virtual_joint
- removed joint qbhand2m_manipulation_joint
- removed joint qbhand2m_middle_distal_joint
- removed joint qbhand2m_middle_distal_virtual_joint
- removed joint qbhand2m_middle_knuckle_joint
- removed joint qbhand2m_middle_middle_joint
- removed joint qbhand2m_middle_middle_virtual_joint
- removed joint qbhand2m_middle_proximal_joint
- removed joint qbhand2m_middle_proximal_virtual_joint
- removed joint qbhand2m_motor_1_joint
- removed joint qbhand2m_motor_2_joint
- removed joint qbhand2m_palm_fixed_joint
- removed joint qbhand2m_ring_distal_joint
- removed joint qbhand2m_ring_distal_virtual_joint
- removed joint qbhand2m_ring_knuckle_joint
- removed joint qbhand2m_ring_middle_joint
- removed joint qbhand2m_ring_middle_virtual_joint
- removed joint qbhand2m_ring_proximal_joint
- removed joint qbhand2m_ring_proximal_virtual_joint
- removed joint qbhand2m_thumb_distal_joint
- removed joint qbhand2m_thumb_distal_virtual_joint
- removed joint qbhand2m_thumb_knuckle_joint
- removed joint qbhand2m_thumb_proximal_joint
- removed joint qbhand2m_thumb_proximal_virtual_joint
- added joint camera_joint: type fixed, parent camera_support_link, child camera_frame, origin xyz=0.06 0.06 0.02 rpy=0.0872665 0 2.35619
- added joint qbhand2m1_base_fixed_joint: type fixed, parent camera_support_link, child qbhand2m1_base_link, origin xyz=0 0 0.01 rpy=0 0 2.356194490192345
- added joint qbhand2m1_end_effector_fixed_joint: type fixed, parent qbhand2m1_base_link, child qbhand2m1_end_effector_link, origin xyz=-0.03 0.060 0.142 rpy=-1.57 0 0
- added joint qbhand2m1_index_distal_joint: type revolute, parent qbhand2m1_index_middle_link, child qbhand2m1_index_distal_virtual_link, origin xyz=0.009 0 0 rpy=0 0 0, axis 0 0 -1, limit lower=0.0 upper=0.785 effort=100 velocity=100, mimic joint=qbhand2m1_synergy_joint multiplier=0.785
- added joint qbhand2m1_index_distal_virtual_joint: type revolute, parent qbhand2m1_index_distal_virtual_link, child qbhand2m1_index_distal_link, origin xyz=0.013 0 0 rpy=0 0 0, axis 0 0 -1, limit lower=0.0 upper=0.785 effort=100 velocity=100, mimic joint=qbhand2m1_index_distal_joint multiplier=1.0
- added joint qbhand2m1_index_knuckle_joint: type revolute, parent qbhand2m1_palm_link, child qbhand2m1_index_knuckle_link, origin xyz=-0.02 -0.007 0.014 rpy=0 0 1.57, axis 0 0 -1, limit lower=-0.524 upper=0.524 effort=100 velocity=100, mimic joint=qbhand2m1_synergy_joint multiplier=-0.2
- added joint qbhand2m1_index_middle_joint: type revolute, parent qbhand2m1_index_proximal_link, child qbhand2m1_index_middle_virtual_link, origin xyz=0.017 0 0 rpy=0 0 0, axis 0 0 -1, limit lower=0.0 upper=0.785 effort=100 velocity=100, mimic joint=qbhand2m1_synergy_joint multiplier=0.785
- added joint qbhand2m1_index_middle_virtual_joint: type revolute, parent qbhand2m1_index_middle_virtual_link, child qbhand2m1_index_middle_link, origin xyz=0.013 0 0 rpy=0 0 0, axis 0 0 -1, limit lower=0.0 upper=0.785 effort=100 velocity=100, mimic joint=qbhand2m1_index_middle_joint multiplier=1.0
- added joint qbhand2m1_index_proximal_joint: type revolute, parent qbhand2m1_index_knuckle_link, child qbhand2m1_index_proximal_virtual_link, origin xyz=0.009 0 0 rpy=1.57 0 0, axis 0 0 -1, limit lower=0.0 upper=0.785 effort=100 velocity=100, mimic joint=qbhand2m1_synergy_joint multiplier=0.785
- added joint qbhand2m1_index_proximal_virtual_joint: type revolute, parent qbhand2m1_index_proximal_virtual_link, child qbhand2m1_index_proximal_link, origin xyz=0.013 0 0 rpy=0 0 0, axis 0 0 -1, limit lower=0.0 upper=0.785 effort=100 velocity=100, mimic joint=qbhand2m1_index_proximal_joint multiplier=1.0
- added joint qbhand2m1_little_distal_joint: type revolute, parent qbhand2m1_little_middle_link, child qbhand2m1_little_distal_virtual_link, origin xyz=0.009 0 0 rpy=0 0 0, axis 0 0 -1, limit lower=0.0 upper=0.785 effort=100 velocity=100, mimic joint=qbhand2m1_synergy_joint multiplier=0.785
- added joint qbhand2m1_little_distal_virtual_joint: type revolute, parent qbhand2m1_little_distal_virtual_link, child qbhand2m1_little_distal_link, origin xyz=0.013 0 0 rpy=0 0 0, axis 0 0 -1, limit lower=0.0 upper=0.785 effort=100 velocity=100, mimic joint=qbhand2m1_little_distal_joint multiplier=1.0
- added joint qbhand2m1_little_knuckle_joint: type revolute, parent qbhand2m1_palm_link, child qbhand2m1_little_knuckle_link, origin xyz=0.04 -0.012 0.014 rpy=0 0 1.57, axis 0 0 -1, limit lower=-0.524 upper=0.524 effort=100 velocity=100, mimic joint=qbhand2m1_synergy_joint multiplier=0.4
- added joint qbhand2m1_little_middle_joint: type revolute, parent qbhand2m1_little_proximal_link, child qbhand2m1_little_middle_virtual_link, origin xyz=0.009 0 0 rpy=0 0 0, axis 0 0 -1, limit lower=0.0 upper=0.785 effort=100 velocity=100, mimic joint=qbhand2m1_synergy_joint multiplier=0.785
- added joint qbhand2m1_little_middle_virtual_joint: type revolute, parent qbhand2m1_little_middle_virtual_link, child qbhand2m1_little_middle_link, origin xyz=0.013 0 0 rpy=0 0 0, axis 0 0 -1, limit lower=0.0 upper=0.785 effort=100 velocity=100, mimic joint=qbhand2m1_little_middle_joint multiplier=1.0
- added joint qbhand2m1_little_proximal_joint: type revolute, parent qbhand2m1_little_knuckle_link, child qbhand2m1_little_proximal_virtual_link, origin xyz=0.009 0 0 rpy=1.57 0 0, axis 0 0 -1, limit lower=0.0 upper=0.785 effort=100 velocity=100, mimic joint=qbhand2m1_synergy_joint multiplier=0.785
- added joint qbhand2m1_little_proximal_virtual_joint: type revolute, parent qbhand2m1_little_proximal_virtual_link, child qbhand2m1_little_proximal_link, origin xyz=0.013 0 0 rpy=0 0 0, axis 0 0 -1, limit lower=0.0 upper=0.785 effort=100 velocity=100, mimic joint=qbhand2m1_little_proximal_joint multiplier=1.0
- added joint qbhand2m1_manipulation_joint: type revolute, parent qbhand2m1_palm_link, child qbhand2m1_manipulation_tendon_virtual_link, origin xyz=0 0 0 rpy=0 0 0, axis 0 0 1, limit lower=-1.0 upper=1.0 effort=100 velocity=100
- added joint qbhand2m1_middle_distal_joint: type revolute, parent qbhand2m1_middle_middle_link, child qbhand2m1_middle_distal_virtual_link, origin xyz=0.009 0 0 rpy=0 0 0, axis 0 0 -1, limit lower=0.0 upper=0.785 effort=100 velocity=100, mimic joint=qbhand2m1_synergy_joint multiplier=0.785
- added joint qbhand2m1_middle_distal_virtual_joint: type revolute, parent qbhand2m1_middle_distal_virtual_link, child qbhand2m1_middle_distal_link, origin xyz=0.013 0 0 rpy=0 0 0, axis 0 0 -1, limit lower=0.0 upper=0.785 effort=100 velocity=100, mimic joint=qbhand2m1_middle_distal_joint multiplier=1.0
- added joint qbhand2m1_middle_knuckle_joint: type revolute, parent qbhand2m1_palm_link, child qbhand2m1_middle_knuckle_link, origin xyz=0 0 0.014 rpy=0 0 1.57, axis 0 0 -1, limit lower=-0.524 upper=0.524 effort=100 velocity=100, mimic joint=qbhand2m1_synergy_joint multiplier=0.0
- added joint qbhand2m1_middle_middle_joint: type revolute, parent qbhand2m1_middle_proximal_link, child qbhand2m1_middle_middle_virtual_link, origin xyz=0.017 0 0 rpy=0 0 0, axis 0 0 -1, limit lower=0.0 upper=0.785 effort=100 velocity=100, mimic joint=qbhand2m1_synergy_joint multiplier=0.785
- added joint qbhand2m1_middle_middle_virtual_joint: type revolute, parent qbhand2m1_middle_middle_virtual_link, child qbhand2m1_middle_middle_link, origin xyz=0.013 0 0 rpy=0 0 0, axis 0 0 -1, limit lower=0.0 upper=0.785 effort=100 velocity=100, mimic joint=qbhand2m1_middle_middle_joint multiplier=1.0
- added joint qbhand2m1_middle_proximal_joint: type revolute, parent qbhand2m1_middle_knuckle_link, child qbhand2m1_middle_proximal_virtual_link, origin xyz=0.009 0 0 rpy=1.57 0 0, axis 0 0 -1, limit lower=0.0 upper=0.785 effort=100 velocity=100, mimic joint=qbhand2m1_synergy_joint multiplier=0.785
- added joint qbhand2m1_middle_proximal_virtual_joint: type revolute, parent qbhand2m1_middle_proximal_virtual_link, child qbhand2m1_middle_proximal_link, origin xyz=0.013 0 0 rpy=0 0 0, axis 0 0 -1, limit lower=0.0 upper=0.785 effort=100 velocity=100, mimic joint=qbhand2m1_middle_proximal_joint multiplier=1.0
- added joint qbhand2m1_motor_1_joint: type revolute, parent qbhand2m1_palm_link, child qbhand2m1_motor_1_tendon_virtual_link, origin xyz=0 0 0 rpy=0 0 0, axis 0 0 1, limit lower=0 upper=1.0 effort=100 velocity=100
- added joint qbhand2m1_motor_2_joint: type revolute, parent qbhand2m1_palm_link, child qbhand2m1_motor_2_tendon_virtual_link, origin xyz=0 0 0 rpy=0 0 0, axis 0 0 1, limit lower=0 upper=1.0 effort=100 velocity=100
- added joint qbhand2m1_palm_fixed_joint: type fixed, parent qbhand2m1_base_link, child qbhand2m1_palm_link, origin xyz=-0.0045 0.0145 0.144 rpy=1.57 0 0
- added joint qbhand2m1_ring_distal_joint: type revolute, parent qbhand2m1_ring_middle_link, child qbhand2m1_ring_distal_virtual_link, origin xyz=0.009 0 0 rpy=0 0 0, axis 0 0 -1, limit lower=0.0 upper=0.785 effort=100 velocity=100, mimic joint=qbhand2m1_synergy_joint multiplier=0.785
- added joint qbhand2m1_ring_distal_virtual_joint: type revolute, parent qbhand2m1_ring_distal_virtual_link, child qbhand2m1_ring_distal_link, origin xyz=0.013 0 0 rpy=0 0 0, axis 0 0 -1, limit lower=0.0 upper=0.785 effort=100 velocity=100, mimic joint=qbhand2m1_ring_distal_joint multiplier=1.0
- added joint qbhand2m1_ring_knuckle_joint: type revolute, parent qbhand2m1_palm_link, child qbhand2m1_ring_knuckle_link, origin xyz=0.02 -0.007 0.014 rpy=0 0 1.57, axis 0 0 -1, limit lower=-0.524 upper=0.524 effort=100 velocity=100, mimic joint=qbhand2m1_synergy_joint multiplier=0.2
- added joint qbhand2m1_ring_middle_joint: type revolute, parent qbhand2m1_ring_proximal_link, child qbhand2m1_ring_middle_virtual_link, origin xyz=0.017 0 0 rpy=0 0 0, axis 0 0 -1, limit lower=0.0 upper=0.785 effort=100 velocity=100, mimic joint=qbhand2m1_synergy_joint multiplier=0.785
- added joint qbhand2m1_ring_middle_virtual_joint: type revolute, parent qbhand2m1_ring_middle_virtual_link, child qbhand2m1_ring_middle_link, origin xyz=0.013 0 0 rpy=0 0 0, axis 0 0 -1, limit lower=0.0 upper=0.785 effort=100 velocity=100, mimic joint=qbhand2m1_ring_middle_joint multiplier=1.0
- added joint qbhand2m1_ring_proximal_joint: type revolute, parent qbhand2m1_ring_knuckle_link, child qbhand2m1_ring_proximal_virtual_link, origin xyz=0.009 0 0 rpy=1.57 0 0, axis 0 0 -1, limit lower=0.0 upper=0.785 effort=100 velocity=100, mimic joint=qbhand2m1_synergy_joint multiplier=0.785
- added joint qbhand2m1_ring_proximal_virtual_joint: type revolute, parent qbhand2m1_ring_proximal_virtual_link, child qbhand2m1_ring_proximal_link, origin xyz=0.013 0 0 rpy=0 0 0, axis 0 0 -1, limit lower=0.0 upper=0.785 effort=100 velocity=100, mimic joint=qbhand2m1_ring_proximal_joint multiplier=1.0
- added joint qbhand2m1_synergy_joint: type revolute, parent qbhand2m1_palm_link, child qbhand2m1_synergy_tendon_virtual_link, origin xyz=0 0 0 rpy=0 0 0, axis 0 0 1, limit lower=0.0 upper=1.0 effort=100 velocity=100
- added joint qbhand2m1_thumb_distal_joint: type revolute, parent qbhand2m1_thumb_proximal_link, child qbhand2m1_thumb_distal_virtual_link, origin xyz=0.009 0 0 rpy=0 0 0, axis 0 0 -1, limit lower=0.0 upper=0.785 effort=100 velocity=100, mimic joint=qbhand2m1_synergy_joint multiplier=0.785
- added joint qbhand2m1_thumb_distal_virtual_joint: type revolute, parent qbhand2m1_thumb_distal_virtual_link, child qbhand2m1_thumb_distal_link, origin xyz=0.013 0 0 rpy=0 0 0, axis 0 0 -1, limit lower=0.0 upper=0.785 effort=100 velocity=100, mimic joint=qbhand2m1_thumb_distal_joint multiplier=1.0
- added joint qbhand2m1_thumb_knuckle_joint: type revolute, parent qbhand2m1_palm_link, child qbhand2m1_thumb_knuckle_link, origin xyz=-0.044 -0.0465 -0.002 rpy=-1.57 3.14 0.0, axis 0 0 -1, limit lower=0.0 upper=1.571 effort=100 velocity=100, mimic joint=qbhand2m1_synergy_joint multiplier=2.542
- added joint qbhand2m1_thumb_proximal_joint: type revolute, parent qbhand2m1_thumb_knuckle_link, child qbhand2m1_thumb_proximal_virtual_link, origin xyz=0.0255 -0.0038 -0.00012 rpy=-1.1415 0.0 0.0, axis 0 0 -1, limit lower=0.0 upper=0.785 effort=100 velocity=100, mimic joint=qbhand2m1_synergy_joint multiplier=0.785
- added joint qbhand2m1_thumb_proximal_virtual_joint: type revolute, parent qbhand2m1_thumb_proximal_virtual_link, child qbhand2m1_thumb_proximal_link, origin xyz=0.013 0 0 rpy=0 0 0, axis 0 0 -1, limit lower=0.0 upper=0.785 effort=100 velocity=100, mimic joint=qbhand2m1_thumb_proximal_joint multiplier=1.0

File: panda_qb_description/urdf/pandaqb_robot.xacro (robot description, xacro)
@@ -10,5 +10,5 @@
       <!-- Import the QB Hand and connect it to the created link -->
       <xacro:include filename="$(find qb_hand_description)/urdf/qbhand.utils.xacro"/>
-      <xacro:build_hand_2m_from_yaml configuration="qbhand_right" namespace="qbhand2m" parent="camera_support">
+      <xacro:build_hand_2m_from_yaml configuration="qbhand_right" namespace="qbhand2m1" parent="camera_support">
         <origin xyz="0 0 0.01" rpy="0 0 ${3*pi/4}"/>
       </xacro:build_hand_2m_from_yaml>
