Commit message: hand eye calibration launchfile

File: panda_qb_description/urdf/camera_support.xacro (robot description, xacro)
@@ -28,3 +28,10 @@
     </inertial>
   </link>
+  <!-- Gazebo requires a joint to a link called "world" for statically mounted robots -->
+  <link name="camera_frame" />
+  <joint name="camera_joint" type="fixed">
+    <origin xyz="0.1 0 0.1" rpy="0 0 0" />
+    <parent link="camera_support_link" />
+    <child  link="camera_frame" />
+  </joint>
 </robot>

Commit message: added camera parameters and accurate camera frame

File: panda_qb_description/urdf/camera_support.xacro (robot description, xacro)
@@ -31,5 +31,5 @@
   <link name="camera_frame" />
   <joint name="camera_joint" type="fixed">
-    <origin xyz="0.1 0 0.1" rpy="0 0 0" />
+    <origin xyz="0.06 0.06 0.02" rpy="0.0872665 0 2.35619" />
     <parent link="camera_support_link" />
     <child  link="camera_frame" />

Commit message: Removed all non-necessary files in pandaqb_movegroup_control

File: panda_qb_description/urdf/camera_support.xacro (robot description, xacro)
@@ -10,5 +10,5 @@
       <origin rpy="0 0 -${pi/4}" xyz="-0.051 0.00 -0.009"/>
       <geometry>
-        <mesh filename="package://pandaqb_movegroup_control/meshes/camera_support.stl" scale="0.001 0.001 0.001"/>
+        <mesh filename="package://panda_qb_description/meshes/camera_support.stl" scale="0.001 0.001 0.001"/>
       </geometry>
       <material name="gray">
@@ -19,5 +19,5 @@
       <origin rpy="0 0 -${pi/4}" xyz="-0.051 0.00 -0.009"/>
       <geometry>
-        <mesh filename="package://pandaqb_movegroup_control/meshes/camera_support.stl" scale="0.001 0.001 0.001"/>
+        <mesh filename="package://panda_qb_description/meshes/camera_support.stl" scale="0.001 0.001 0.001"/>
       </geometry>
     </collision>

Commit message: Send the robot to a previous pose depending on the grasp orientation

File: panda_qb_description/urdf/camera_support.xacro (robot description, xacro)
@@ -8,5 +8,5 @@
   <link name="camera_support_link">
     <visual>
-      <origin rpy="0 0 -${pi/4}" xyz="-0.051 0.00 -0.009"/>
+      <origin rpy="0 0 -${pi/2}" xyz="-0.036 0.036 -0.009"/>
       <geometry>
         <mesh filename="package://panda_qb_description/meshes/camera_support.stl" scale="0.001 0.001 0.001"/>
@@ -17,5 +17,5 @@
     </visual>
     <collision>
-      <origin rpy="0 0 -${pi/4}" xyz="-0.051 0.00 -0.009"/>
+      <origin rpy="0 0 -${pi/2}" xyz="-0.036 0.036 -0.009"/>
       <geometry>
         <mesh filename="package://panda_qb_description/meshes/camera_support.stl" scale="0.001 0.001 0.001"/>
@@ -23,5 +23,5 @@
     </collision>
     <inertial>
-      <origin rpy="0 0 -${pi/4}" xyz="-0.051 0.00 -0.009"/>
+      <origin rpy="0 0 -${pi/2}" xyz="-0.036 0.036 -0.009"/>
       <mass value="0.1"/>
       <inertia ixx="0.001" ixy="0.001" ixz="0.001" iyy="0.001" iyz="0.001" izz="0.001" />

File: panda_qb_description/urdf/pandaqb_robot.xacro (robot description, xacro)
@@ -11,5 +11,5 @@
       <xacro:include filename="$(find qb_hand_description)/urdf/qbhand.utils.xacro"/>
       <xacro:build_hand_2m_from_yaml configuration="qbhand_right" namespace="qbhand2m1" parent="camera_support">
-        <origin xyz="0 0 0.01" rpy="0 0 ${3*pi/4}"/>
+        <origin xyz="0 0 0.01" rpy="0 0 ${pi/2}"/>
       </xacro:build_hand_2m_from_yaml>
     </xacro:if>

Commit message: Register success in grasps

File: panda_qb_description/urdf/camera_support.xacro (robot description, xacro)
@@ -8,7 +8,7 @@
   <link name="camera_support_link">
     <visual>
-      <origin rpy="0 0 -${pi/2}" xyz="-0.036 0.036 -0.009"/>
+      <origin rpy="0 0 -${pi/2}" xyz="0 0 0.00"/>
       <geometry>
-        <mesh filename="package://panda_qb_description/meshes/camera_support.stl" scale="0.001 0.001 0.001"/>
+        <mesh filename="package://panda_qb_description/meshes/gripper_cam_support.stl" scale="0.001 0.001 0.001"/>
       </geometry>
       <material name="gray">
@@ -17,11 +17,11 @@
     </visual>
     <collision>
-      <origin rpy="0 0 -${pi/2}" xyz="-0.036 0.036 -0.009"/>
+      <origin rpy="0 0 -${pi/2}" xyz="0 0 0.00"/>
       <geometry>
-        <mesh filename="package://panda_qb_description/meshes/camera_support.stl" scale="0.001 0.001 0.001"/>
+        <mesh filename="package://panda_qb_description/meshes/gripper_cam_support.stl" scale="0.001 0.001 0.001"/>
       </geometry>
     </collision>
     <inertial>
-      <origin rpy="0 0 -${pi/2}" xyz="-0.036 0.036 -0.009"/>
+      <origin rpy="0 0 -${pi/2}" xyz="0 0 0.00"/>
       <mass value="0.1"/>
       <inertia ixx="0.001" ixy="0.001" ixz="0.001" iyy="0.001" iyz="0.001" izz="0.001" />

File: panda_qb_description/urdf/panda_gripper.xacro (robot description, xacro)
@@ -13,5 +13,5 @@
           arm_id="$(arg arm_id)"
           rpy="0 0 0"
-          xyz="0 0 0.011"
+          xyz="0 0 0.015"
           connected_to="camera_support_link"
           safety_distance="0.03"

Commit message: solved camera pose and tf out of range vision problems

File: panda_qb_description/urdf/camera_support.xacro (robot description, xacro)
@@ -30,4 +30,5 @@
   <link name="camera_frame" />
   <joint name="camera_joint" type="fixed">
+    <!-- <origin xyz="-0.0414091 -0.0579333 0.0614579" rpy="-0.019865 0.0305123 -0.0144474 0.999233" /> -->
     <origin xyz="0.06 0.06 0.02" rpy="0.0872665 0 2.35619" />
     <parent link="camera_support_link" />

File: panda_qb_description/urdf/pandaqb_robot.xacro (robot description, xacro)
@@ -11,5 +11,5 @@
       <xacro:include filename="$(find qb_hand_description)/urdf/qbhand.utils.xacro"/>
       <xacro:build_hand_2m_from_yaml configuration="qbhand_right" namespace="qbhand2m1" parent="qb_hand_wrist">
-        <origin xyz="0.018 0.0 0.068" rpy="${pi/2} 0 ${pi/2}"/>
+        <origin xyz="0.018 0.0 0.063" rpy="${pi/2} 0 ${pi/2}"/>
       </xacro:build_hand_2m_from_yaml>
     </xacro:if>

File: panda_qb_description/urdf/qb_hand_wrist.xacro (robot description, xacro)
@@ -8,5 +8,5 @@
   <link name="qb_hand_wrist_link">
     <visual>
-      <origin rpy="0 0 ${pi/2}" xyz="0.0 0.0 -0.007"/>
+      <origin rpy="0 0 ${-pi/2}" xyz="0.0 0.0 -0.007"/>
       <geometry>
         <mesh filename="package://panda_qb_description/meshes/qb_hand_wrist.stl" scale="0.001 0.001 0.001"/>
@@ -17,5 +17,5 @@
     </visual>
     <collision>
-      <origin rpy="0 0 ${pi/2}" xyz="0.0 0.0 -0.007"/> <!-- -${pi/2} -->
+      <origin rpy="0 0 ${-pi/2}" xyz="0.0 0.0 -0.007"/> <!-- -${pi/2} -->
       <geometry>
         <mesh filename="package://panda_qb_description/meshes/qb_hand_wrist.stl" scale="0.001 0.001 0.001"/>
@@ -23,14 +23,15 @@
     </collision>
     <inertial>
-      <origin rpy="0 0 ${pi/2}" xyz="0.0 0.0 -0.007"/>
+      <origin rpy="0 0 ${-pi/2}" xyz="0.0 0.0 -0.007"/>
       <mass value="0.1"/>
       <inertia ixx="0.001" ixy="0.001" ixz="0.001" iyy="0.001" iyz="0.001" izz="0.001" />
     </inertial>
   </link>
-  <link name="camera_frame" />
+  <!-- <link name="camera_frame" />
   <joint name="camera_joint" type="fixed">
+    <origin xyz="-0.0414091 -0.0579333 0.0614579" rpy="-0.0389014 0.0615907 -0.0277165" />
     <origin xyz="0.06 0.06 0.02" rpy="0.0872665 0 2.35619" />
     <parent link="qb_hand_wrist_link" />
     <child  link="camera_frame" />
-  </joint>
+  </joint> -->
 </robot>

Commit message: updates for the franka eef

File: panda_qb_description/urdf/camera_support.xacro (robot description, xacro)
@@ -8,5 +8,5 @@
   <link name="camera_support_link">
     <visual>
-      <origin rpy="0 0 -${pi/2}" xyz="0 0 0.00"/>
+      <origin rpy="0 0 ${pi/4}" xyz="0 0 0.00"/>
       <geometry>
         <mesh filename="package://panda_qb_description/meshes/gripper_cam_support.stl" scale="0.001 0.001 0.001"/>
@@ -17,5 +17,5 @@
     </visual>
     <collision>
-      <origin rpy="0 0 -${pi/2}" xyz="0 0 0.00"/>
+      <origin rpy="0 0 ${pi/4}" xyz="0 0 0.00"/>
       <geometry>
         <mesh filename="package://panda_qb_description/meshes/gripper_cam_support.stl" scale="0.001 0.001 0.001"/>
@@ -23,12 +23,13 @@
     </collision>
     <inertial>
-      <origin rpy="0 0 -${pi/2}" xyz="0 0 0.00"/>
+      <origin rpy="0 0 ${pi/4}" xyz="0 0 0.00"/>
       <mass value="0.1"/>
       <inertia ixx="0.001" ixy="0.001" ixz="0.001" iyy="0.001" iyz="0.001" izz="0.001" />
     </inertial>
   </link>
-  <!-- <joint name="camera_joint" type="fixed">
-    <origin xyz="-0.041387 -0.0627379 0.0525437" rpy="3.08447 -3.11784 3.10978" />
-    <parent link="panda_link8" />
+  <!-- <link name="camera_frame" />
+  <joint name="camera_joint" type="fixed">
+    <origin xyz="-0.0152599 0.0628288 0.0195069" rpy="2.96575 -2.9721 0.76305"/>
+    <parent link="camera_support_link" />
     <child  link="camera_frame" />
   </joint> -->

File: panda_qb_description/urdf/panda_gripper.xacro (robot description, xacro)
@@ -12,5 +12,5 @@
       <xacro:franka_hand
           arm_id="$(arg arm_id)"
-          rpy="0 0 0"
+          rpy="0 0 -${pi/4}"
           xyz="0 0 0.015"
           connected_to="camera_support_link"

File: panda_qb_description/urdf/pandaqb_robot.xacro (robot description, xacro)
@@ -15,5 +15,5 @@
     <link name="pinch_link" />
     <joint name="pinch_joint" type="fixed">
-      <origin xyz="-0.0 -0.014 0.022" rpy="0 0 0.523598775" />
+      <origin xyz="-0.013 -0.002 0.033" rpy="0 0 0.523598775" />
       <parent link="qbhand2m1_end_effector_link" />
       <child  link="pinch_link" />
