Commit message: New moveit config using the wrist

File: panda_qb_description/urdf/pandaqb_robot.xacro (robot description, xacro)
@@ -6,10 +6,10 @@
     <xacro:include filename="$(find franka_description)/robots/common/franka_arm.xacro" />
     <xacro:franka_arm arm_id="panda" safety_distance="0.03" gazebo="$(arg gazebo)" joint_limits="${joint_limits}"/>
-    <xacro:include filename="$(find panda_qb_description)/urdf/camera_support.xacro"/>
+    <xacro:include filename="$(find panda_qb_description)/urdf/qb_hand_wrist.xacro"/>
     <xacro:if value="$(arg hand)">
       <!-- Import the QB Hand and connect it to the created link -->
       <xacro:include filename="$(find qb_hand_description)/urdf/qbhand.utils.xacro"/>
-      <xacro:build_hand_2m_from_yaml configuration="qbhand_right" namespace="qbhand2m1" parent="camera_support">
-        <origin xyz="0 0 0.01" rpy="0 0 ${pi/2}"/>
+      <xacro:build_hand_2m_from_yaml configuration="qbhand_right" namespace="qbhand2m1" parent="qb_hand_wrist">
+        <origin xyz="0.018 0.0 0.058" rpy="${pi/2} 0 ${pi/2}"/>
       </xacro:build_hand_2m_from_yaml>
     </xacro:if>

Commit message: EEF controller to select between gripper or qb hand

File: panda_qb_description/urdf/pandaqb_robot.xacro (robot description, xacro)
@@ -11,5 +11,5 @@
       <xacro:include filename="$(find qb_hand_description)/urdf/qbhand.utils.xacro"/>
       <xacro:build_hand_2m_from_yaml configuration="qbhand_right" namespace="qbhand2m1" parent="qb_hand_wrist">
-        <origin xyz="0.018 0.0 0.058" rpy="${pi/2} 0 ${pi/2}"/>
+        <origin xyz="0.018 0.0 0.068" rpy="${pi/2} 0 ${pi/2}"/>
       </xacro:build_hand_2m_from_yaml>
     </xacro:if>

File: panda_qb_description/urdf/qb_hand_wrist.xacro (robot description, xacro)
@@ -8,5 +8,5 @@
   <link name="qb_hand_wrist_link">
     <visual>
-      <origin rpy="0 0 ${-pi/2}" xyz="0.0 0.0 -0.007"/>
+      <origin rpy="0 0 ${pi/2}" xyz="0.0 0.0 -0.007"/>
       <geometry>
         <mesh filename="package://panda_qb_description/meshes/qb_hand_wrist.stl" scale="0.001 0.001 0.001"/>
@@ -17,5 +17,5 @@
     </visual>
     <collision>
-      <origin rpy="0 0 ${-pi/2}" xyz="0.0 0.0 0.0"/> <!-- -${pi/2} -->
+      <origin rpy="0 0 ${pi/2}" xyz="0.0 0.0 -0.007"/> <!-- -${pi/2} -->
       <geometry>
         <mesh filename="package://panda_qb_description/meshes/qb_hand_wrist.stl" scale="0.001 0.001 0.001"/>
@@ -23,5 +23,5 @@
     </collision>
     <inertial>
-      <origin rpy="0 0 ${-pi/2}" xyz="0.0 0.0 0.0"/>
+      <origin rpy="0 0 ${pi/2}" xyz="0.0 0.0 -0.007"/>
       <mass value="0.1"/>
       <inertia ixx="0.001" ixy="0.001" ixz="0.001" iyy="0.001" iyz="0.001" izz="0.001" />

Commit message: the system is precise for pinch but darknet still not working for all objects

File: panda_qb_description/urdf/pandaqb_robot.xacro (robot description, xacro)
@@ -13,4 +13,10 @@
         <origin xyz="0.018 0.0 0.063" rpy="${pi/2} 0 ${pi/2}"/>
       </xacro:build_hand_2m_from_yaml>
+    <link name="pinch_link" />
+    <joint name="pinch_joint" type="fixed">
+      <origin xyz="-0.005 -0.017 0.030" rpy="0.174532925 0 0.523598775" />
+      <parent link="qbhand2m1_end_effector_link" />
+      <child  link="pinch_link" />
+    </joint>
     </xacro:if>
   </xacro:macro>

File: panda_qb_description/urdf/qb_hand_wrist.xacro (robot description, xacro)
@@ -28,10 +28,9 @@
     </inertial>
   </link>
-  <!-- <link name="camera_frame" />
+  <link name="camera_frame" />
   <joint name="camera_joint" type="fixed">
-    <origin xyz="-0.0414091 -0.0579333 0.0614579" rpy="-0.0389014 0.0615907 -0.0277165" />
-    <origin xyz="0.06 0.06 0.02" rpy="0.0872665 0 2.35619" />
+    <origin xyz="-0.0371711 -0.0595898 0.0627352" rpy="3.10255 2.99161 3.10566" />
     <parent link="qb_hand_wrist_link" />
     <child  link="camera_frame" />
-  </joint> -->
+  </joint>
 </robot>

Commit message: update

File: panda_qb_description/urdf/pandaqb_robot.xacro (robot description, xacro)
@@ -15,7 +15,13 @@
     <link name="pinch_link" />
     <joint name="pinch_joint" type="fixed">
-      <origin xyz="-0.005 -0.017 0.030" rpy="0.174532925 0 0.523598775" />
+      <origin xyz="-0.003 -0.015 0.022" rpy="0.0872665 0 0.523598775" />
       <parent link="qbhand2m1_end_effector_link" />
       <child  link="pinch_link" />
+    </joint>
+    <link name="power_link" />
+    <joint name="power_joint" type="fixed">
+      <origin xyz="0.05 -0.02 0.0" rpy="0 0 0.523598775" />
+      <parent link="qbhand2m1_end_effector_link" />
+      <child  link="power_link" />
     </joint>
     </xacro:if>

Commit message: ready for the experiment (almost)

File: panda_qb_description/urdf/pandaqb_robot.xacro (robot description, xacro)
@@ -21,5 +21,5 @@
     <link name="power_link" />
     <joint name="power_joint" type="fixed">
-      <origin xyz="0.05 -0.02 0.0" rpy="0 0 0.523598775" />
+      <origin xyz="0.01 -0.02 0.0" rpy="0 0 0.523598775" />
       <parent link="qbhand2m1_end_effector_link" />
       <child  link="power_link" />

Commit message: finger collision checking

File: panda_qb_description/urdf/pandaqb_robot.xacro (robot description, xacro)
@@ -15,5 +15,5 @@
     <link name="pinch_link" />
     <joint name="pinch_joint" type="fixed">
-      <origin xyz="-0.003 -0.015 0.022" rpy="0.0872665 0 0.523598775" />
+      <origin xyz="-0.003 -0.012 0.022" rpy="0.0872665 0 0.523598775" />
       <parent link="qbhand2m1_end_effector_link" />
       <child  link="pinch_link" />

Commit message: almost ready for the experiments

File: panda_qb_description/urdf/pandaqb_robot.xacro (robot description, xacro)
@@ -15,5 +15,5 @@
     <link name="pinch_link" />
     <joint name="pinch_joint" type="fixed">
-      <origin xyz="-0.003 -0.012 0.022" rpy="0.0872665 0 0.523598775" />
+      <origin xyz="0.007 -0.009 0.022" rpy="0.0872665 0 0.523598775" />
       <parent link="qbhand2m1_end_effector_link" />
       <child  link="pinch_link" />

Commit message: fskjds

File: panda_qb_description/urdf/pandaqb_robot.xacro (robot description, xacro)
@@ -21,5 +21,5 @@
     <link name="power_link" />
     <joint name="power_joint" type="fixed">
-      <origin xyz="0.02 -0.02 -0.005" rpy="0 0 0.523598775" />
+      <origin xyz="0.02 -0.02 -0.005" rpy="0 0 0" />
       <parent link="qbhand2m1_end_effector_link" />
       <child  link="power_link" />

File: panda_qb_description/urdf/qb_hand_wrist.xacro (robot description, xacro)
@@ -28,9 +28,9 @@
     </inertial>
   </link>
-  <link name="camera_frame" />
+  <!-- <link name="camera_frame" />
   <joint name="camera_joint" type="fixed">
     <origin xyz="-0.041387 -0.0627379 0.0525437" rpy="3.08447 -3.11784 3.10978" />
     <parent link="panda_link8" />
     <child  link="camera_frame" />
-  </joint>
+  </joint> -->
 </robot>
